File: 1URack_8Input_AB_2Output_Mixer.sch (KiCad schematic (older format))
At the start: 48 parts

Commit message: First Commit
Connections:
- wire segments 145 -> 184
Other:
- moved on the sheet: C_BYNEG1, C_BYPOS1, C_OABY1, C_OABY2, FADER1, FADER2, FADER3, FADER4, FADER5, FADER6, FADER7, FADER8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

Commit message: Updates
Parts:
- removed FADER1, FADER2, FADER3, FADER4, FADER5, FADER6, FADER7, FADER8: A50K, symbol NPOT
- added FADER1, FADER2, FADER3, FADER4, FADER5, FADER6, FADER7, FADER8: B50K, Bourn_PTL_Slider:Slider_PTL20_LED_35MM, symbol NPOT_LED
- added R_LED1, R_LED2, R_LED3, R_LED4, R_LED5, R_LED6, R_LED7, R_LED8: 560R, Resistors_SMD:R_0805_HandSoldering, symbol R
- C_BYNEG1, C_BYPOS1, C_OABY1, C_OABY2: footprint (none) -> Capacitors_SMD:C_0805_HandSoldering
- J_POWER1: footprint (none) -> Pin_Headers:Pin_Header_Angled_2x05_Pitch2.54mm
- R_IN1, R_IN2, R_IN3, R_IN4, R_IN5, R_IN6, R_IN7, R_IN8, R_OUTA1, R_OUTA2, R_OUTA3, R_OUTB1, R_OUTB2, R_OUTB3: footprint (none) -> Resistors_SMD:R_0805_HandSoldering
- SW_AB1, SW_AB2, SW_AB3, SW_AB4, SW_AB5, SW_AB6, SW_AB7, SW_AB8: footprint (none) -> custom_sw:SW_SPDT_W6.86MM_L12.7MM_P4.8MM_D2MM
Other:
- moved on the sheet: J_IN1

Commit message: Updates
Parts:
- removed U_OUT1, U_OUT2: TL074, symbol TL074
- added C_OUT2_NEG1, C_OUT2_POS1: 100nF, Capacitors_SMD:C_0805_HandSoldering, symbol C
- added U_OUT1, U_OUT2: TL072_InversedInputs, symbol TL072_InversedInputs
- renumbered C_OABY2 to C_OUT1_NEG1, C_OABY1 to C_OUT1_POS1, R_OUTA1 to R_OUT1_1, R_OUTA2 to R_OUT1_2, R_OUTA3 to R_OUT1_3, R_OUTB1 to R_OUT2_1, R_OUTB2 to R_OUT2_2, R_OUTB3 to R_OUT2_3
Connections:
- wire segments 184 -> 235
Other:
- moved on the sheet: C_OUT1_NEG1, C_OUT1_POS1

Commit message: Updates
Parts:
- R_IN1, R_IN2, R_IN3, R_IN4, R_IN5, R_IN6, R_IN7, R_IN8: value 100K -> 5K6
Changed lines of the file:
@@
 P 3750 4875
 F 0 "R_IN1" V 3830 4875 50  0000 C CNN
-F 1 "100K" V 3750 4875 50  0000 C CNN
+F 1 "5K6" V 3750 4875 50  0000 C CNN
 F 2 "Resistors_SMD:R_0805_HandSoldering" V 3680 4875 50  0001 C CNN
 F 3 "" H 3750 4875 50  0001 C CNN
@@
 P 3750 6475
 F 0 "R_IN2" V 3830 6475 50  0000 C CNN
-F 1 "100K" V 3750 6475 50  0000 C CNN
+F 1 "5K6" V 3750 6475 50  0000 C CNN
 F 2 "Resistors_SMD:R_0805_HandSoldering" V 3680 6475 50  0001 C CNN
 F 3 "" H 3750 6475 50  0001 C CNN
@@
 P 3750 8125
 F 0 "R_IN3" V 3830 8125 50  0000 C CNN
-F 1 "100K" V 3750 8125 50  0000 C CNN
+F 1 "5K6" V 3750 8125 50  0000 C CNN
 F 2 "Resistors_SMD:R_0805_HandSoldering" V 3680 8125 50  0001 C CNN
 F 3 "" H 3750 8125 50  0001 C CNN
@@
 P 3750 9775
 F 0 "R_IN4" V 3830 9775 50  0000 C CNN
-F 1 "100K" V 3750 9775 50  0000 C CNN
+F 1 "5K6" V 3750 9775 50  0000 C CNN
 F 2 "Resistors_SMD:R_0805_HandSoldering" V 3680 9775 50  0001 C CNN
 F 3 "" H 3750 9775 50  0001 C CNN
@@
 P 3750 11425
 F 0 "R_IN5" V 3830 11425 50  0000 C CNN
-F 1 "100K" V 3750 11425 50  0000 C CNN
+F 1 "5K6" V 3750 11425 50  0000 C CNN
 F 2 "Resistors_SMD:R_0805_HandSoldering" V 3680 11425 50  0001 C CNN
 F 3 "" H 3750 11425 50  0001 C CNN
@@
 P 3750 13025
 F 0 "R_IN6" V 3830 13025 50  0000 C CNN
-F 1 "100K" V 3750 13025 50  0000 C CNN
+F 1 "5K6" V 3750 13025 50  0000 C CNN
 F 2 "Resistors_SMD:R_0805_HandSoldering" V 3680 13025 50  0001 C CNN
 F 3 "" H 3750 13025 50  0001 C CNN
@@
 P 3750 14675
 F 0 "R_IN7" V 3830 14675 50  0000 C CNN
-F 1 "100K" V 3750 14675 50  0000 C CNN
+F 1 "5K6" V 3750 14675 50  0000 C CNN
 F 2 "Resistors_SMD:R_0805_HandSoldering" V 3680 14675 50  0001 C CNN
 F 3 "" H 3750 14675 50  0001 C CNN
@@
 P 3750 16325
 F 0 "R_IN8" V 3830 16325 50  0000 C CNN
-F 1 "100K" V 3750 16325 50  0000 C CNN
+F 1 "5K6" V 3750 16325 50  0000 C CNN
 F 2 "Resistors_SMD:R_0805_HandSoldering" V 3680 16325 50  0001 C CNN
 F 3 "" H 3750 16325 50  0001 C CNN

Commit message: update
- Recalculated gain values on opamps
Parts:
- removed R_OUT1_3, R_OUT2_3: 100K, Resistors_SMD:R_0805_HandSoldering, symbol R
- added VR_ChanA_OAout_Rf1, VR_ChanB_OAout_Rf1: B100K, symbol NPOT
- FADER1, FADER2, FADER3, FADER4, FADER5, FADER6, FADER7, FADER8: value B50K -> B100K
- R_ChanAB_OAin_Rin1: renamed from R_IN1; value 5K6 -> 10K
- R_ChanAB_OAin_Rin2: renamed from R_IN2; value 5K6 -> 10K
- R_ChanAB_OAin_Rin3: renamed from R_IN3; value 5K6 -> 10K
- R_ChanAB_OAin_Rin4: renamed from R_IN4; value 5K6 -> 10K
- R_ChanAB_OAin_Rin5: renamed from R_IN5; value 5K6 -> 10K
- R_ChanAB_OAin_Rin6: renamed from R_IN6; value 5K6 -> 10K
- R_ChanAB_OAin_Rin7: renamed from R_IN7; value 5K6 -> 10K
- R_ChanAB_OAin_Rin8: renamed from R_IN8; value 5K6 -> 10K
- R_ChanA_OAin_Rf1: renamed from R_OUT1_1; value 100K -> 10K
- R_ChanA_OAout_Rin1: renamed from R_OUT1_2; value 100K -> 56K
- R_ChanB_OAin_Rf1: renamed from R_OUT2_1; value 100K -> 10K
- R_ChanB_OAout_Rin1: renamed from R_OUT2_2; value 100K -> 56K
- renumbered U_OUT1 to ChanA_OA1, U_OUT2 to ChanB_OA1, J_OUT1 to J_ChanA_out1, J_OUT2 to J_ChanB_out1
Connections:
- net at ChanA_OA1.6 (-), R_ChanA_OAout_Rin1.1: now also VR_ChanA_OAout_Rf1.3
- net at ChanA_OA1.7, J_ChanA_out1.1: now also VR_ChanA_OAout_Rf1.1, VR_ChanA_OAout_Rf1.2
- net at ChanB_OA1.6 (-), R_ChanB_OAout_Rin1.1: now also VR_ChanB_OAout_Rf1.3
- net at ChanB_OA1.7, J_ChanB_out1.1: now also VR_ChanB_OAout_Rf1.1, VR_ChanB_OAout_Rf1.2
Other:
- note added: "GAIN = -1.79\n20vpp"
- note added: "GAIN = 1 (unity)\n10vpp\n"
- moved on the sheet: ChanA_OA1A, ChanA_OA1B, ChanB_OA1A, ChanB_OA1B, FADER1, FADER2, FADER3, FADER4, FADER5, FADER6, FADER7, FADER8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

Commit message: update
Parts:
- removed J_ChanA_out1, J_ChanB_out1, J_IN1, J_IN2, J_IN3, J_IN4, J_IN5, J_IN6, J_IN7, J_IN8: Audio-Jack-2, symbol Audio-Jack-2
- removed J_POWER1: Conn_02x05_Top_Bottom, Pin_Headers:Pin_Header_Angled_2x05_Pitch2.54mm, symbol Conn_02x05_Top_Bottom
- removed Q_POL1: Q_PMOS_GDS, symbol Q_PMOS_GDS
- removed SW_AB1, SW_AB2, SW_AB3, SW_AB4, SW_AB5, SW_AB6, SW_AB7, SW_AB8: SW_SP3T, custom_sw:SW_SPDT_W6.86MM_L12.7MM_P4.8MM_D2MM, symbol SW_SP3T
- added J_ChanA_out1, J_ChanB_out1, J_IN1, J_IN2, J_IN3, J_IN4, J_IN5, J_IN6, J_IN7, J_IN8: Audio-JackMono_Tip3_Sw2_Slv1, ThonkiConn_3:Conn_3.5mmJackMono_Vertical_PJ301BM, symbol Audio-JackMono_Tip3_Sw2_Slv1
- added J_PWR1: EurorackPowerConnector_2x5Pin, symbol EurorackPowerConnector_2x5Pin
- added SW_AB1, SW_AB2, SW_AB3, SW_AB4, SW_AB5, SW_AB6, SW_AB7, SW_AB8: SW_SPDT, DailywellSwitches:Dailywell_SPDT, symbol SW_SPDT
- U_ChanA_OA1: renamed from ChanA_OA1; footprint (none) -> SMD_Packages:SOIC-8-N
- U_ChanA_OA1: renamed from U_OUT2; footprint (none) -> SMD_Packages:SOIC-8-N
- U_ChanB_OA1: renamed from ChanB_OA1; footprint (none) -> SMD_Packages:SOIC-8-N
- U_ChanB_OA1: renamed from U_OUT1; footprint (none) -> SMD_Packages:SOIC-8-N
- VR_ChanA_OAout_Rf1, VR_ChanB_OAout_Rf1: footprint (none) -> Bourn_PTL_Slider:Slider_PTL20_LED_35MM
- renumbered C_OUT2_NEG1 to C_ChanA_NEGBY1, C_OUT2_POS1 to C_ChanA_POSBY1, C_OUT1_NEG1 to C_ChanB_BYNEG1, C_OUT1_POS1 to C_ChanB_BYPOS1, C_BYNEG1 to C_PW_BYNEG1, C_BYPOS1 to C_PW_BYPOS1, FADER1 to VR_FADER1, FADER2 to VR_FADER2, FADER3 to VR_FADER3, FADER4 to VR_FADER4, FADER5 to VR_FADER5, FADER6 to VR_FADER6, FADER7 to VR_FADER7, FADER8 to VR_FADER8
Connections:
- net 12VIN+ is gone; now on net 12V+: C_PW_BYPOS1.1
- net 12V+: now also J_PWR1.1 (Pin_1)
- net 12V-: now also J_PWR1.9 (Pin_9)
- net GND: now also J_ChanA_out1.1, J_ChanA_out1.2, J_ChanB_out1.1, J_ChanB_out1.2, J_IN1.1, J_IN1.2, J_IN2.1, J_IN2.2, J_IN3.1, J_IN3.2, J_IN4.1, J_IN4.2, J_IN5.1, J_IN5.2, J_IN6.1, J_IN6.2, J_IN7.1, J_IN7.2, J_IN8.1, J_IN8.2, J_PWR1.5 (Pin_5)
- net at VR_FADER1.1: now also J_IN1.3
- net at R_ChanAB_OAin_Rin1.1: now also SW_AB1.2 (B)
- net at R_ChanA_OAin_Rf1.2, U_ChanA_OA1.2 (-): now also SW_AB1.1 (A), SW_AB2.1 (A), SW_AB3.1 (A), SW_AB4.1 (A), SW_AB5.1 (A), SW_AB6.1 (A), SW_AB7.1 (A), SW_AB8.1 (A)
- net at R_ChanB_OAin_Rf1.2, U_ChanB_OA1.2 (-): now also SW_AB1.3 (C), SW_AB2.3 (C), SW_AB3.3 (C), SW_AB4.3 (C), SW_AB5.3 (C), SW_AB6.3 (C), SW_AB7.3 (C), SW_AB8.3 (C)
- net at U_ChanA_OA1.7, VR_ChanA_OAout_Rf1.1, VR_ChanA_OAout_Rf1.2: now also J_ChanA_out1.3
- net at U_ChanB_OA1.7, VR_ChanB_OAout_Rf1.1, VR_ChanB_OAout_Rf1.2: now also J_ChanB_out1.3
- net at VR_FADER2.1: now also J_IN2.3
- net at R_ChanAB_OAin_Rin2.1: now also SW_AB2.2 (B)
- net at VR_FADER3.1: now also J_IN3.3
- net at R_ChanAB_OAin_Rin3.1: now also SW_AB3.2 (B)
- net at VR_FADER4.1: now also J_IN4.3
- net at R_ChanAB_OAin_Rin4.1: now also SW_AB4.2 (B)
- net at VR_FADER5.1: now also J_IN5.3
- net at R_ChanAB_OAin_Rin5.1: now also SW_AB5.2 (B)
- net at VR_FADER6.1: now also J_IN6.3
- net at R_ChanAB_OAin_Rin6.1: now also SW_AB6.2 (B)
- net at VR_FADER7.1: now also J_IN7.3
- net at R_ChanAB_OAin_Rin7.1: now also SW_AB7.2 (B)
- net at VR_FADER8.1: now also J_IN8.3
- net at R_ChanAB_OAin_Rin8.1: now also SW_AB8.2 (B)
- no-connect marks 15 -> 7
Other:
- moved on the sheet: C_ChanA_NEGBY1, C_ChanA_POSBY1, C_ChanB_BYNEG1, C_ChanB_BYPOS1, C_PW_BYNEG1, C_PW_BYPOS1

Commit message: updates
Parts:
- J_PWR1: footprint (none) -> Pin_Headers:Pin_Header_Straight_2x05_Pitch2.54mm
- R_ChanA_OAout_Rin1, R_ChanB_OAout_Rin1: value 56K -> 25K
- VR_ChanA_OAout_Rf1, VR_ChanB_OAout_Rf1, VR_FADER1, VR_FADER3, VR_FADER5, VR_FADER6, VR_FADER7, VR_FADER8: value B100K -> B50K
- VR_FADER2, VR_FADER4: value B100K -> B5K
Other:
- note added: "All VR_ChanX_OAout:\nCC = +6dB (x2)\nCCW = 0vpp"
- note added: "All VR_Faders:\nCC = Unity 0dB\nCCW = 0vpp\n"
- note added: "For +6dB gain (x2):\n50K -> B100K\n22K -> B50K\n5K -> B10K"
- note removed: "GAIN = -1.79\n20vpp"
- note removed: "GAIN = 1 (unity)\n10vpp\n"
Changed lines of the file:
@@
 P 7975 1400
 F 0 "R_ChanA_OAout_Rin1" V 8055 1400 50  0000 C CNN
-F 1 "56K" V 7975 1400 50  0000 C CNN
+F 1 "25K" V 7975 1400 50  0000 C CNN
 F 2 "Resistors_SMD:R_0805_HandSoldering" V 7905 1400 50  0001 C CNN
 F 3 "" H 7975 1400 50  0001 C CNN
@@
 	0    1    1    0
 $EndComp
-Text Label 5600 3450 1    60   ~ 0
-GND
-Text Label 8000 3450 1    60   ~ 0
-GND
-Text Label 9900 3450 1    60   ~ 0
+Text Label 5600 3300 1    60   ~ 0
+GND
+Text Label 8000 3300 1    60   ~ 0
+GND
+Text Label 9900 3300 1    60   ~ 0
 GND
 $Comp
@@
 P 8000 4000
 F 0 "R_ChanB_OAout_Rin1" V 8080 4000 50  0000 C CNN
-F 1 "56K" V 8000 4000 50  0000 C CNN
+F 1 "25K" V 8000 4000 50  0000 C CNN
 F 2 "Resistors_SMD:R_0805_HandSoldering" V 7930 4000 50  0001 C CNN
 F 3 "" H 8000 4000 50  0001 C CNN
@@
 	6200 2650 5600 2650
 Wire Wire Line
-	5600 2650 5600 3450
+	5600 2650 5600 3300
 Wire Wire Line
 	8750 2750 8000 2750
 Wire Wire Line
-	8000 2750 8000 3450
+	8000 2750 8000 3300
 Connection ~ 9900 2650
 Wire Wire Line
 	10025 2750 9900 2750
 Wire Wire Line
-	9900 2750 9900 3450
+	9900 2750 9900 3300
 Wire Wire Line
 	5200 4000 6375 4000
@@
 P 2900 4875
 F 0 "VR_FADER1" H 3075 5150 50  0000 C CNN
-F 1 "B100K" H 3075 5075 50  0000 C CNN
+F 1 "B50K" H 3075 5075 50  0000 C CNN
 F 2 "Bourn_PTL_Slider:Slider_PTL20_LED_35MM" H 2900 4875 50  0001 C CNN
 F 3 "" H 2900 4875 50  0001 C CNN
@@
 P 2900 6475
 F 0 "VR_FADER2" H 3150 6725 50  0000 C CNN
-F 1 "B100K" H 3150 6625 50  0000 C CNN
+F 1 "B5K" H 3150 6625 50  0000 C CNN
 F 2 "Bourn_PTL_Slider:Slider_PTL20_LED_35MM" H 2900 6475 50  0001 C CNN
 F 3 "" H 2900 6475 50  0001 C CNN
@@
 P 2900 8125
 F 0 "VR_FADER3" H 3150 8400 50  0000 C CNN
-F 1 "B100K" H 3150 8300 50  0000 C CNN
+F 1 "B50K" H 3150 8300 50  0000 C CNN
 F 2 "Bourn_PTL_Slider:Slider_PTL20_LED_35MM" H 2900 8125 50  0001 C CNN
 F 3 "" H 2900 8125 50  0001 C CNN
@@
 P 2900 9775
 F 0 "VR_FADER4" H 3125 10050 50  0000 C CNN
-F 1 "B100K" H 3125 9975 50  0000 C CNN
+F 1 "B5K" H 3125 9975 50  0000 C CNN
 F 2 "Bourn_PTL_Slider:Slider_PTL20_LED_35MM" H 2900 9775 50  0001 C CNN
 F 3 "" H 2900 9775 50  0001 C CNN
@@
 P 2900 11425
 F 0 "VR_FADER5" H 3125 11650 50  0000 C CNN
-F 1 "B100K" H 3125 11575 50  0000 C CNN
+F 1 "B50K" H 3125 11575 50  0000 C CNN
 F 2 "Bourn_PTL_Slider:Slider_PTL20_LED_35MM" H 2900 11425 50  0001 C CNN
 F 3 "" H 2900 11425 50  0001 C CNN
@@
 P 2900 13025
 F 0 "VR_FADER6" H 3100 13300 50  0000 C CNN
-F 1 "B100K" H 3100 13200 50  0000 C CNN
+F 1 "B50K" H 3100 13200 50  0000 C CNN
 F 2 "Bourn_PTL_Slider:Slider_PTL20_LED_35MM" H 2900 13025 50  0001 C CNN
 F 3 "" H 2900 13025 50  0001 C CNN
@@
 P 2925 14675
 F 0 "VR_FADER7" H 3200 14925 50  0000 C CNN
-F 1 "B100K" H 3175 14850 50  0000 C CNN
+F 1 "B50K" H 3175 14850 50  0000 C CNN
 F 2 "Bourn_PTL_Slider:Slider_PTL20_LED_35MM" H 2925 14675 50  0001 C CNN
 F 3 "" H 2925 14675 50  0001 C CNN
@@
 P 2925 16325
 F 0 "VR_FADER8" H 3175 16600 50  0000 C CNN
-F 1 "B100K" H 3175 16525 50  0000 C CNN
+F 1 "B50K" H 3175 16525 50  0000 C CNN
 F 2 "Bourn_PTL_Slider:Slider_PTL20_LED_35MM" H 2925 16325 50  0001 C CNN
 F 3 "" H 2925 16325 50  0001 C CNN
@@
 P 9150 1400
 F 0 "VR_ChanA_OAout_Rf1" V 8975 1400 50  0000 C CNN
-F 1 "B100K" V 9050 1400 50  0000 C CNN
+F 1 "B50K" V 9050 1400 50  0000 C CNN
 F 2 "Bourn_PTL_Slider:Slider_PTL20_LED_35MM" H 9150 1400 50  0001 C CNN
 F 3 "" H 9150 1400 50  0001 C CNN
@@
 	9450 1150 9450 1400
 Connection ~ 9450 1400
-Text Notes 5975 1850 0    60   ~ 0
-GAIN = 1 (unity)\n10vpp\n
-Text Notes 8875 2050 0    60   ~ 0
-GAIN = -1.79\n20vpp
 $Comp
 L NPOT VR_ChanB_OAout_Rf1
@@
 P 9100 4000
 F 0 "VR_ChanB_OAout_Rf1" V 8925 4000 50  0000 C CNN
-F 1 "B100K" V 9000 4000 50  0000 C CNN
+F 1 "B50K" V 9000 4000 50  0000 C CNN
 F 2 "Bourn_PTL_Slider:Slider_PTL20_LED_35MM" H 9100 4000 50  0001 C CNN
 F 3 "" H 9100 4000 50  0001 C CNN
@@
 $EndComp
 Wire Wire Line
-	10425 2850 10425 3075
-Wire Wire Line
-	10425 3075 9900 3075
-Connection ~ 9900 3075
+	10425 2850 10425 2975
+Wire Wire Line
+	10425 2975 9900 2975
+Connection ~ 9900 2975
 Wire Wire Line
 	10400 5375 10400 5475
@@
 F 0 "J_PWR1" H 7600 8825 50  0000 C CNN
 F 1 "EurorackPowerConnector_2x5Pin" H 7725 8150 50  0000 C CNN
-F 2 "" H 7550 8525 50  0001 C CNN
+F 2 "Pin_Headers:Pin_Header_Straight_2x05_Pitch2.54mm" H 7550 8525 50  0001 C CNN
 F 3 "" H 7550 8525 50  0001 C CNN
 	1    7550 8525
 	-1   0    0    -1
 $EndComp
+Text Notes 9950 1050 0    60   ~ 0
+For +6dB gain (x2):\n50K -> B100K\n22K -> B50K\n5K -> B10K
+Text Notes 8725 950  0    60   ~ 0
+All VR_ChanX_OAout:\nCC = +6dB (x2)\nCCW = 0vpp
+Text Notes 3025 4400 0    60   ~ 0
+All VR_Faders:\nCC = Unity 0dB\nCCW = 0vpp\n
 $EndSCHEMATC

Commit message: First draft board layout
Parts:
- removed VR_ChanA_OAout_Rf1, VR_ChanB_OAout_Rf1: B50K, Bourn_PTL_Slider:Slider_PTL20_LED_35MM, symbol NPOT
- added R_ChanA_OAout1, R_ChanB_OAout1: 1K, Resistors_SMD:R_0805_HandSoldering, symbol R
- added VR_ChanA_OAout_Rf1, VR_ChanB_OAout_Rf1: B50K, Bourn_PTL_Slider:Slider_PTL20_LED_35MM, symbol NPOT_LED
- J_ChanA_out1, J_ChanB_out1, J_IN1, J_IN2, J_IN3, J_IN4, J_IN5, J_IN6, J_IN7, J_IN8: footprint ThonkiConn_3:Conn_3.5mmJackMono_Vertical_PJ301BM -> ThonkiConn_3:Conn_3.5mmJackMono_Vertical_PJ301M-12
Connections:
- net 12V+: now also VR_ChanA_OAout_Rf1.4, VR_ChanB_OAout_Rf1.4
- net GND: now also R_ChanA_OAout1.2, R_ChanB_OAout1.2
- net at R_ChanA_OAout_Rin1.1, U_ChanA_OA1.6 (-): now also VR_ChanA_OAout_Rf1.3
- net at R_ChanB_OAout_Rin1.1, U_ChanB_OA1.6 (-): now also VR_ChanB_OAout_Rf1.3
- net at J_ChanA_out1.3, U_ChanA_OA1.7: now also VR_ChanA_OAout_Rf1.1, VR_ChanA_OAout_Rf1.2
- net at J_ChanB_out1.3, U_ChanB_OA1.7: now also VR_ChanB_OAout_Rf1.1, VR_ChanB_OAout_Rf1.2
- new net: R_ChanA_OAout1.1, VR_ChanA_OAout_Rf1.5
- new net: R_ChanB_OAout1.1, VR_ChanB_OAout_Rf1.5
Other:
- moved on the sheet: R_ChanA_OAin_Rf1, R_ChanA_OAout_Rin1, R_ChanB_OAin_Rf1, R_ChanB_OAout_Rin1, U_ChanA_OA1A, U_ChanA_OA1B, U_ChanB_OA1A, U_ChanB_OA1B
