File: 1URack_8Input_AB_2Output_Mixer.sch (KiCad schematic (older format))
At the start: 59 parts

Commit message: second draft
Parts:
- R_ChanA_OAout_Rin1, R_ChanB_OAout_Rin1: value 25K -> 22K
- R_LED1, R_LED2, R_LED3, R_LED4, R_LED5, R_LED6, R_LED7, R_LED8: value 560R -> 2K2
Connections:
- wire segments 215 -> 273
Other:
- note added: "All VR_ChanX_OAout:\nFull CW = +6dBv (10vpp -> 20vpp)\n1/4 CCW = +4dBv (10vpp -> 16vpp)\n1/2 CCW = 0dBv (unity)\n3/4 CCW = -12dBv (10vpp -> 2.5vpp)\nFull CCW = 0vpp"
- note added: "All VR_Faders:\nFull CW = 0dB (unity)\n1\4 CCW = -6dBv (10vpp -> 5vpp)\n1\2 CCW= -12dBv (10vpp -> 2.5vpp)\n3\4 CCW= -20dBv (10vpp -> 1vpp)\nFull CCW = infinity (0vpp)\n"
- note added: "For +6dB gain (x2):\nRin -> Rfb\n50K -> B100K\n22K -> B50K\n5K -> B10K"
- note removed: "All VR_ChanX_OAout:\nCC = +6dB (x2)\nCCW = 0vpp"
- note removed: "All VR_Faders:\nCC = Unity 0dB\nCCW = 0vpp\n"
- note removed: "For +6dB gain (x2):\n50K -> B100K\n22K -> B50K\n5K -> B10K"
- moved on the sheet: VR_ChanA_OAout_Rf1

Commit message: third draft
Connections:
- wire segments 273 -> 215
Other:
- note added: "1 x TL072\n= 9mA"
- note added: "12v / 2200\n= 5.5mA"
Changed lines of the file:
@@
 	1600 4725 1775 4725
 Wire Wire Line
-	1775 4725 1775 5050
-Wire Wire Line
-	1775 5050 1775 5475
-Wire Wire Line
-	2900 5025 2900 5475
-Wire Wire Line
-	2900 5475 2900 5750
-Wire Wire Line
-	1775 5475 2725 5475
-Wire Wire Line
-	2725 5475 2900 5475
+	1775 4725 1775 5475
+Wire Wire Line
+	2900 5025 2900 5750
+Wire Wire Line
+	1775 5475 2900 5475
 Connection ~ 2900 5475
 Wire Wire Line
@@
 	4750 4775 4450 4775
 Wire Wire Line
-	4450 4975 5200 4975
-Wire Wire Line
-	5200 4975 5900 4975
+	4450 4975 5900 4975
 Wire Wire Line
 	4750 2450 5700 2450
@@
 	4750 1400 5650 1400
 Wire Wire Line
-	5950 1400 6550 1400
-Wire Wire Line
-	6550 1400 7100 1400
+	5950 1400 7100 1400
 Wire Wire Line
 	6550 2550 6550 1400
@@
 	8025 2550 8025 1400
 Wire Wire Line
-	7400 1400 8025 1400
-Wire Wire Line
-	8025 1400 8600 1400
-Wire Wire Line
-	8900 1400 9050 1400
-Wire Wire Line
-	9050 1400 9900 1400
+	7400 1400 8600 1400
+Wire Wire Line
+	8900 1400 9900 1400
 Wire Wire Line
 	9900 1400 9900 2650
 Wire Wire Line
-	8950 2650 9900 2650
-Wire Wire Line
-	9900 2650 10025 2650
+	8950 2650 10025 2650
 Connection ~ 8025 1400
 Wire Wire Line
@@
 	10025 2750 9900 2750
 Wire Wire Line
-	9900 2750 9900 2975
-Wire Wire Line
-	9900 2975 9900 3300
+	9900 2750 9900 3300
 Wire Wire Line
 	5200 4000 6075 4000
 Wire Wire Line
-	6375 4000 6725 4000
-Wire Wire Line
-	6725 4000 7200 4000
+	6375 4000 7200 4000
 Wire Wire Line
 	6725 5075 6725 4000
@@
 	8050 5075 8050 4000
 Wire Wire Line
-	7500 4000 8050 4000
-Wire Wire Line
-	8050 4000 8775 4000
-Wire Wire Line
-	9075 4000 9275 4000
-Wire Wire Line
-	9275 4000 9875 4000
+	7500 4000 8775 4000
+Wire Wire Line
+	9075 4000 9875 4000
 Wire Wire Line
 	9875 4000 9875 5175
 Connection ~ 8050 4000
 Wire Wire Line
-	5200 4000 5200 4975
-Wire Wire Line
-	5200 4975 5200 6575
-Wire Wire Line
-	5200 6575 5200 8225
-Wire Wire Line
-	5200 8225 5200 9875
-Wire Wire Line
-	5200 9875 5200 11525
-Wire Wire Line
-	5200 11525 5200 13125
-Wire Wire Line
-	5200 13125 5200 14775
-Wire Wire Line
-	5200 14775 5200 16425
+	5200 4000 5200 16425
 Wire Wire Line
 	6500 5075 6725 5075
@@
 	8050 5075 8650 5075
 Wire Wire Line
-	9250 5175 9875 5175
-Wire Wire Line
-	9875 5175 10000 5175
+	9250 5175 10000 5175
 Connection ~ 5200 4975
 Wire Wire Line
@@
 	10000 5275 9875 5275
 Wire Wire Line
-	9875 5275 9875 5475
-Wire Wire Line
-	9875 5475 9875 5775
-Wire Wire Line
-	10075 9800 10075 10075
-Wire Wire Line
-	10075 10075 10075 10800
-Wire Wire Line
-	10075 11600 10075 12175
-Wire Wire Line
-	10075 12175 10075 12675
+	9875 5275 9875 5775
+Wire Wire Line
+	10075 9800 10075 10800
+Wire Wire Line
+	10075 11600 10075 12675
 Connection ~ 4750 4775
 Wire Wire Line
-	7750 8525 9050 8525
-Wire Wire Line
-	9050 8525 10025 8525
+	7750 8525 10025 8525
 Wire Wire Line
 	7750 8725 8150 8725
 Wire Wire Line
-	8150 8975 9050 8975
-Wire Wire Line
-	9050 8975 10025 8975
-Wire Wire Line
-	8150 8125 9050 8125
-Wire Wire Line
-	9050 8125 10025 8125
+	8150 8975 10025 8975
+Wire Wire Line
+	8150 8125 10025 8125
 Wire Wire Line
 	8150 8125 8150 8325
@@
 $EndComp
 Wire Wire Line
-	9050 8475 9050 8525
-Wire Wire Line
-	9050 8525 9050 8575
+	9050 8475 9050 8575
 Connection ~ 9050 8125
 Wire Wire Line
@@
 	1600 6325 1775 6325
 Wire Wire Line
-	1775 6325 1775 6650
-Wire Wire Line
-	1775 6650 1775 7075
-Wire Wire Line
-	2900 6625 2900 7075
-Wire Wire Line
-	2900 7075 2900 7350
-Wire Wire Line
-	1775 7075 2725 7075
-Wire Wire Line
-	2725 7075 2900 7075
+	1775 6325 1775 7075
+Wire Wire Line
+	2900 6625 2900 7350
+Wire Wire Line
+	1775 7075 2900 7075
 Connection ~ 2900 7075
 Wire Wire Line
@@
 	1600 7975 1775 7975
 Wire Wire Line
-	1775 7975 1775 8350
-Wire Wire Line
-	1775 8350 1775 8725
-Wire Wire Line
-	2900 8275 2900 8725
-Wire Wire Line
-	2900 8725 2900 9000
-Wire Wire Line
-	1775 8725 2725 8725
-Wire Wire Line
-	2725 8725 2900 8725
+	1775 7975 1775 8725
+Wire Wire Line
+	2900 8275 2900 9000
+Wire Wire Line
+	1775 8725 2900 8725
 Connection ~ 2900 8725
 Wire Wire Line
@@
 	1600 9625 1775 9625
 Wire Wire Line
-	1775 9625 1775 10000
-Wire Wire Line
-	1775 10000 1775 10375
-Wire Wire Line
-	2900 9925 2900 10375
-Wire Wire Line
-	2900 10375 2900 10650
-Wire Wire Line
-	1775 10375 2725 10375
-Wire Wire Line
-	2725 10375 2900 10375
+	1775 9625 1775 10375
+Wire Wire Line
+	2900 9925 2900 10650
+Wire Wire Line
+	1775 10375 2900 10375
 Connection ~ 2900 10375
 Wire Wire Line
@@
 	1600 11275 1775 11275
 Wire Wire Line
-	1775 11275 1775 11650
-Wire Wire Line
-	1775 11650 1775 12025
-Wire Wire Line
-	2900 11575 2900 12025
-Wire Wire Line
-	2900 12025 2900 12300
-Wire Wire Line
-	1775 12025 2725 12025
-Wire Wire Line
-	2725 12025 2900 12025
+	1775 11275 1775 12025
+Wire Wire Line
+	2900 11575 2900 12300
+Wire Wire Line
+	1775 12025 2900 12025
 Connection ~ 2900 12025
 Wire Wire Line
@@
 	1600 12875 1775 12875
 Wire Wire Line
-	1775 12875 1775 13250
-Wire Wire Line
-	1775 13250 1775 13625
-Wire Wire Line
-	2900 13175 2900 13625
-Wire Wire Line
-	2900 13625 2900 13900
-Wire Wire Line
-	1775 13625 2725 13625
-Wire Wire Line
-	2725 13625 2900 13625
+	1775 12875 1775 13625
+Wire Wire Line
+	2900 13175 2900 13900
+Wire Wire Line
+	1775 13625 2900 13625
 Connection ~ 2900 13625
 Wire Wire Line
@@
 	1625 14525 1800 14525
 Wire Wire Line
-	1800 14525 1800 14900
-Wire Wire Line
-	1800 14900 1800 15275
-Wire Wire Line
-	2925 14825 2925 15275
-Wire Wire Line
-	2925 15275 2925 15550
-Wire Wire Line
-	1800 15275 2750 15275
-Wire Wire Line
-	2750 15275 2925 15275
+	1800 14525 1800 15275
+Wire Wire Line
+	2925 14825 2925 15550
+Wire Wire Line
+	1800 15275 2925 15275
 Connection ~ 2925 15275
 Wire Wire Line
@@
 	1625 16175 1800 16175
 Wire Wire Line
-	1800 16175 1800 16550
-Wire Wire Line
-	1800 16550 1800 16925
-Wire Wire Line
-	2925 16475 2925 16925
-Wire Wire Line
-	2925 16925 2925 17200
-Wire Wire Line
-	1800 16925 2750 16925
-Wire Wire Line
-	2750 16925 2925 16925
+	1800 16175 1800 16925
+Wire Wire Line
+	2925 16475 2925 17200
+Wire Wire Line
+	1800 16925 2925 16925
 Connection ~ 2925 16925
 Wire Wire Line
@@
 	2750 16550 2750 16475
 Wire Wire Line
-	4750 1400 4750 2450
-Wire Wire Line
-	4750 2450 4750 4775
-Wire Wire Line
-	4750 4775 4750 6375
-Wire Wire Line
-	4750 6375 4750 8025
-Wire Wire Line
-	4750 8025 4750 9675
-Wire Wire Line
-	4750 9675 4750 11325
-Wire Wire Line
-	4750 11325 4750 12925
-Wire Wire Line
-	4750 12925 4750 14575
-Wire Wire Line
-	4750 14575 4750 16225
+	4750 1400 4750 16225
 Wire Wire Line
 	4750 16225 4450 16225
@@
 12V-
 Wire Wire Line
-	7475 9800 7475 10075
-Wire Wire Line
-	7475 10075 7475 10775
-Wire Wire Line
-	7475 11575 7475 12175
-Wire Wire Line
-	7475 12175 7475 12675
+	7475 9800 7475 10775
+Wire Wire Line
+	7475 11575 7475 12675
 $Comp
 L C C_ChanA_POSBY1
@@
 Text Label 9600 4175 2    60   ~ 0
 12V+
+Text Notes 2000 5125 0    60   ~ 0
+12v / 2200\n= 5.5mA
+Text Notes 7125 4825 0    60   ~ 0
+1 x TL072\n= 9mA
 $EndSCHEMATC

Commit message: updated to Kicad 5
Parts:
- C_ChanA_NEGBY1, C_ChanA_POSBY1, C_ChanB_BYNEG1, C_ChanB_BYPOS1, C_PW_BYNEG1, C_PW_BYPOS1: symbol C -> Device:C
- J_ChanA_out1, J_ChanB_out1, J_IN1, J_IN2, J_IN3, J_IN4, J_IN5, J_IN6, J_IN7, J_IN8: symbol Audio-JackMono_Tip3_Sw2_Slv1 -> Conn_audio-jackmono_tip3_sw2_slv1:Audio-JackMono_Tip3_Sw2_Slv1
- J_PWR1: symbol EurorackPowerConnector_2x5Pin -> EurorackPowerConnector_2x5Pin:EurorackPowerConnector_2x5Pin
- R_ChanAB_OAin_Rin1, R_ChanAB_OAin_Rin2, R_ChanAB_OAin_Rin3, R_ChanAB_OAin_Rin4, R_ChanAB_OAin_Rin5, R_ChanAB_OAin_Rin6, R_ChanAB_OAin_Rin7, R_ChanAB_OAin_Rin8, R_ChanA_OAin_Rf1, R_ChanA_OAout1, R_ChanA_OAout_Rin1, R_ChanB_OAin_Rf1, R_ChanB_OAout1, R_ChanB_OAout_Rin1, R_LED1, R_LED2, R_LED3, R_LED4, R_LED5, R_LED6, R_LED7, R_LED8: symbol R -> Device:R
- SW_AB1, SW_AB2, SW_AB3, SW_AB4, SW_AB5, SW_AB6, SW_AB7, SW_AB8: symbol SW_SPDT -> 1URack_8Input_AB_2Output_Mixer-rescue:SW_SPDT
- U_ChanA_OA1, U_ChanB_OA1: symbol TL072_InversedInputs -> tl072_inversedinputs:TL072_InversedInputs
- VR_ChanA_OAout_Rf1, VR_ChanB_OAout_Rf1, VR_FADER1, VR_FADER2, VR_FADER3, VR_FADER4, VR_FADER5, VR_FADER6, VR_FADER7, VR_FADER8: symbol NPOT_LED -> npot_led:NPOT_LED
Connections:
- wire segments 215 -> 273
