File: _saved_1URack_8Input_AB_2Output_Mixer.sch (KiCad schematic (older format))
At the start: 59 parts

Commit message: second draft
Connections:
- wire segments 215 -> 273
Other:
- note added: "1 x TL072\n= 9mA"
- note added: "12v / 2200\n= 5.5mA"
- note added: "All VR_ChanX_OAout:\nFull CW = +6dBv (10vpp -> 20vpp)\n1/4 CCW = +4dBv (10vpp -> 16vpp)\n1/2 CCW = 0dBv (unity)\n3/4 CCW = -12dBv (10vpp -> 2.5vpp)\nFull CCW = 0vpp"
- note added: "All VR_Faders:\nFull CW = 0dB (unity)\n1\4 CCW = -6dBv (10vpp -> 5vpp)\n1\2 CCW= -12dBv (10vpp -> 2.5vpp)\n3\4 CCW= -20dBv (10vpp -> 1vpp)\nFull CCW = infinity (0vpp)\n"
- note added: "For +6dB gain (x2):\nRin -> Rfb\n50K -> B100K\n22K -> B50K\n5K -> B10K"
- note removed: "All VR_ChanX_OAout:\nCC = +6dB (x2)\nCCW = 0vpp"
- note removed: "All VR_Faders:\nCC = Unity 0dB\nCCW = 0vpp\n"
- note removed: "For +6dB gain (x2):\n50K -> B100K\n22K -> B50K\n5K -> B10K"
- moved on the sheet: VR_ChanA_OAout_Rf1
