File: 1URack_8Input_AB_2Output_Mixer.kicad_pcb (KiCad board)
At the start: 2 copper layers, 478.8 x 43.2 mm, 0 parts

Commit message: update
Parts:
- added C_ChanA_NEGBY1: 100nF, Capacitors_SMD:C_0805_HandSoldering, F.Cu at (377.8, 158.7)
- added C_ChanA_POSBY1: 100nF, Capacitors_SMD:C_0805_HandSoldering, F.Cu at (374.0, 144.8)
- added C_ChanB_BYNEG1: 100nF, Capacitors_SMD:C_0805_HandSoldering, F.Cu at (421.0, 159.4)
- added C_ChanB_BYPOS1: 100nF, Capacitors_SMD:C_0805_HandSoldering, F.Cu at (417.2, 145.4)
- added C_PW_BYNEG1: 100nF, Capacitors_SMD:C_0805_HandSoldering, F.Cu at (457.2, 158.8)
- added C_PW_BYPOS1: 100nF, Capacitors_SMD:C_0805_HandSoldering, F.Cu at (457.2, 146.1)
- added J_ChanA_out1: Audio-JackMono_Tip3_Sw2_Slv1, ThonkiConn_3:Conn_3.5mmJackMono_Vertical_PJ301BM, F.Cu at (388.2, 159.3)
- added J_ChanB_out1: Audio-JackMono_Tip3_Sw2_Slv1, ThonkiConn_3:Conn_3.5mmJackMono_Vertical_PJ301BM, F.Cu at (431.4, 159.4)
- added J_IN1: Audio-JackMono_Tip3_Sw2_Slv1, ThonkiConn_3:Conn_3.5mmJackMono_Vertical_PJ301BM, F.Cu at (59.6, 86.4)
- added J_IN2: Audio-JackMono_Tip3_Sw2_Slv1, ThonkiConn_3:Conn_3.5mmJackMono_Vertical_PJ301BM, F.Cu at (94.0, 86.4)
- added J_IN3: Audio-JackMono_Tip3_Sw2_Slv1, ThonkiConn_3:Conn_3.5mmJackMono_Vertical_PJ301BM, F.Cu at (128.3, 86.4)
- added J_IN4: Audio-JackMono_Tip3_Sw2_Slv1, ThonkiConn_3:Conn_3.5mmJackMono_Vertical_PJ301BM, F.Cu at (162.6, 86.1)
- added J_IN5: Audio-JackMono_Tip3_Sw2_Slv1, ThonkiConn_3:Conn_3.5mmJackMono_Vertical_PJ301BM, F.Cu at (196.8, 86.4)
- added J_IN6: Audio-JackMono_Tip3_Sw2_Slv1, ThonkiConn_3:Conn_3.5mmJackMono_Vertical_PJ301BM, F.Cu at (231.1, 85.8)
- added J_IN7: Audio-JackMono_Tip3_Sw2_Slv1, ThonkiConn_3:Conn_3.5mmJackMono_Vertical_PJ301BM, F.Cu at (265.4, 86.1)
- added J_IN8: Audio-JackMono_Tip3_Sw2_Slv1, ThonkiConn_3:Conn_3.5mmJackMono_Vertical_PJ301BM, F.Cu at (299.7, 85.6)
- added J_PWR1: EurorackPowerConnector_2x5Pin, Pin_Headers:Pin_Header_Straight_2x05_Pitch2.54mm, F.Cu at (465.5, 147.3)
- added R_ChanAB_OAin_Rin1: 10K, Resistors_SMD:R_0805_HandSoldering, F.Cu at (59.6, 96.6)
- added R_ChanAB_OAin_Rin2: 10K, Resistors_SMD:R_0805_HandSoldering, F.Cu at (94.0, 96.5)
- added R_ChanAB_OAin_Rin3: 10K, Resistors_SMD:R_0805_HandSoldering, F.Cu at (128.3, 96.5)
- added R_ChanAB_OAin_Rin4: 10K, Resistors_SMD:R_0805_HandSoldering, F.Cu at (162.6, 96.5)
- added R_ChanAB_OAin_Rin5: 10K, Resistors_SMD:R_0805_HandSoldering, F.Cu at (196.8, 96.5)
- added R_ChanAB_OAin_Rin6: 10K, Resistors_SMD:R_0805_HandSoldering, F.Cu at (231.1, 96.2)
- added R_ChanAB_OAin_Rin7: 10K, Resistors_SMD:R_0805_HandSoldering, F.Cu at (265.4, 96.5)
- added R_ChanAB_OAin_Rin8: 10K, Resistors_SMD:R_0805_HandSoldering, F.Cu at (299.7, 96.5)
- added R_ChanA_OAin_Rf1: 10K, Resistors_SMD:R_0805_HandSoldering, F.Cu at (372.7, 160.0)
- added R_ChanA_OAout_Rin1: 56K, Resistors_SMD:R_0805_HandSoldering, F.Cu at (367.7, 151.8)
- added R_ChanB_OAin_Rf1: 10K, Resistors_SMD:R_0805_HandSoldering, F.Cu at (415.9, 160.7)
- added R_ChanB_OAout_Rin1: 56K, Resistors_SMD:R_0805_HandSoldering, F.Cu at (412.1, 153.0)
- added R_LED1: 560R, Resistors_SMD:R_0805_HandSoldering, F.Cu at (59.6, 115.1)
- added R_LED2: 560R, Resistors_SMD:R_0805_HandSoldering, F.Cu at (94.0, 111.8)
- added R_LED3: 560R, Resistors_SMD:R_0805_HandSoldering, F.Cu at (128.3, 111.8)
- added R_LED4: 560R, Resistors_SMD:R_0805_HandSoldering, F.Cu at (162.6, 111.8)
- added R_LED5: 560R, Resistors_SMD:R_0805_HandSoldering, F.Cu at (196.8, 111.8)
- added R_LED6: 560R, Resistors_SMD:R_0805_HandSoldering, F.Cu at (231.1, 111.5)
- added R_LED7: 560R, Resistors_SMD:R_0805_HandSoldering, F.Cu at (265.4, 111.8)
- added R_LED8: 560R, Resistors_SMD:R_0805_HandSoldering, F.Cu at (299.7, 111.8)
- added SW_AB1: SW_SPDT, DailywellSwitches:Dailywell_SPDT, F.Cu at (59.6, 104.3)
- added SW_AB2: SW_SPDT, DailywellSwitches:Dailywell_SPDT, F.Cu at (94.0, 104.1)
- added SW_AB3: SW_SPDT, DailywellSwitches:Dailywell_SPDT, F.Cu at (128.3, 104.1)
- added SW_AB4: SW_SPDT, DailywellSwitches:Dailywell_SPDT, F.Cu at (162.6, 104.1)
- added SW_AB5: SW_SPDT, DailywellSwitches:Dailywell_SPDT, F.Cu at (196.8, 104.1)
- added SW_AB6: SW_SPDT, DailywellSwitches:Dailywell_SPDT, F.Cu at (231.1, 103.9)
- added SW_AB7: SW_SPDT, DailywellSwitches:Dailywell_SPDT, F.Cu at (265.4, 104.1)
- added SW_AB8: SW_SPDT, DailywellSwitches:Dailywell_SPDT, F.Cu at (299.7, 104.1)
- added U_ChanA_OA1: TL072_InversedInputs, SMD_Packages:SOIC-8-N, F.Cu at (375.9, 151.8)
- added U_ChanB_OA1: TL072_InversedInputs, SMD_Packages:SOIC-8-N, F.Cu at (419.1, 152.4)
- added VR_ChanA_OAout_Rf1: B100K, Bourn_PTL_Slider:Slider_PTL20_LED_35MM, F.Cu at (400.1, 152.1)
- added VR_ChanB_OAout_Rf1: B100K, Bourn_PTL_Slider:Slider_PTL20_LED_35MM, F.Cu at (443.2, 152.1)
- added VR_FADER1: B100K, Bourn_PTL_Slider:Slider_PTL20_LED_35MM, F.Cu at (74.8, 96.5)
- added VR_FADER2: B100K, Bourn_PTL_Slider:Slider_PTL20_LED_35MM, F.Cu at (108.0, 96.5)
- added VR_FADER3: B100K, Bourn_PTL_Slider:Slider_PTL20_LED_35MM, F.Cu at (142.3, 96.5)
- added VR_FADER4: B100K, Bourn_PTL_Slider:Slider_PTL20_LED_35MM, F.Cu at (176.5, 96.5)
- added VR_FADER5: B100K, Bourn_PTL_Slider:Slider_PTL20_LED_35MM, F.Cu at (210.8, 96.5)
- added VR_FADER6: B100K, Bourn_PTL_Slider:Slider_PTL20_LED_35MM, F.Cu at (245.1, 96.2)
- added VR_FADER7: B100K, Bourn_PTL_Slider:Slider_PTL20_LED_35MM, F.Cu at (279.5, 96.5)
- added VR_FADER8: B100K, Bourn_PTL_Slider:Slider_PTL20_LED_35MM, F.Cu at (313.7, 96.5)

Commit message: updates
Parts:
- R_ChanA_OAout_Rin1, R_ChanB_OAout_Rin1: value 56K -> 25K
- VR_ChanA_OAout_Rf1, VR_ChanB_OAout_Rf1, VR_FADER1, VR_FADER3, VR_FADER5, VR_FADER6, VR_FADER7, VR_FADER8: value B100K -> B50K
- VR_FADER2, VR_FADER4: value B100K -> B5K
- moved C_PW_BYNEG1 2.92 mm to (457.2, 155.8), turned to 270 degrees
- moved C_PW_BYPOS1 2.79 mm to (457.2, 148.8), turned to 270 degrees
Connections:
- J_PWR1 pad 10: (no net) -> Net-(J_PWR1-Pad10)
- J_PWR1 pad 2: (no net) -> Net-(J_PWR1-Pad2)
- J_PWR1 pad 3: (no net) -> Net-(J_PWR1-Pad3)
- J_PWR1 pad 4: (no net) -> Net-(J_PWR1-Pad4)
- J_PWR1 pad 6: (no net) -> Net-(J_PWR1-Pad6)
- J_PWR1 pad 7: (no net) -> Net-(J_PWR1-Pad7)
- J_PWR1 pad 8: (no net) -> Net-(J_PWR1-Pad8)
Changed lines of the file:
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@@
     (zones 0)
     (modules 57)
-    (nets 44)
+    (nets 51)
   )
   (page User 599.999 200)
@@
   )
   (setup
-    (last_trace_width 0.75)
+    (last_trace_width 0.25)
     (user_trace_width 0.5)
     (user_trace_width 0.75)
@@
     (pad_to_mask_clearance 0.2)
     (aux_axis_origin 0 0)
-    (visible_elements FFFEFF7F)
+    (visible_elements 7FFFFFFF)
     (pcbplotparams
       (layerselection 0x00030_80000001)
@@
   (net 42 "Net-(R_LED7-Pad1)")
   (net 43 "Net-(R_LED8-Pad1)")
+  (net 44 "Net-(J_PWR1-Pad2)")
+  (net 45 "Net-(J_PWR1-Pad3)")
+  (net 46 "Net-(J_PWR1-Pad4)")
+  (net 47 "Net-(J_PWR1-Pad6)")
+  (net 48 "Net-(J_PWR1-Pad7)")
+  (net 49 "Net-(J_PWR1-Pad8)")
+  (net 50 "Net-(J_PWR1-Pad10)")
   (net_class Default "This is the default net class."
     (clearance 0.2)
@@
     (add_net "Net-(J_IN7-Pad3)")
     (add_net "Net-(J_IN8-Pad3)")
+    (add_net "Net-(J_PWR1-Pad10)")
+    (add_net "Net-(J_PWR1-Pad2)")
+    (add_net "Net-(J_PWR1-Pad3)")
+    (add_net "Net-(J_PWR1-Pad4)")
+    (add_net "Net-(J_PWR1-Pad6)")
+    (add_net "Net-(J_PWR1-Pad7)")
+    (add_net "Net-(J_PWR1-Pad8)")
     (add_net "Net-(R_ChanAB_OAin_Rin1-Pad1)")
     (add_net "Net-(R_ChanAB_OAin_Rin1-Pad2)")
@@
       (effects (font (size 0.5 0.5) (thickness 0.015)))
     )
-    (fp_text value B100K (at 0 -6.604 90) (layer F.Fab)
+    (fp_text value B50K (at 0 -6.604 90) (layer F.Fab)
       (effects (font (size 0.5 0.5) (thickness 0.015)))
     )
@@
       (effects (font (size 0.5 0.5) (thickness 0.015)))
     )
-    (fp_text value B100K (at 0 -6.604 90) (layer F.Fab)
+    (fp_text value B50K (at 0 -6.604 90) (layer F.Fab)
       (effects (font (size 0.5 0.5) (thickness 0.015)))
     )
@@
       (effects (font (size 0.5 0.5) (thickness 0.015)))
     )
-    (fp_text value 56K (at 0 2.1 270) (layer F.Fab)
+    (fp_text value 25K (at 0 2.1 270) (layer F.Fab)
       (effects (font (size 0.5 0.5) (thickness 0.015)))
     )
@@
       (effects (font (size 0.5 0.5) (thickness 0.015)))
     )
-    (fp_text value 56K (at 0 2.1 270) (layer F.Fab)
+    (fp_text value 25K (at 0 2.1 270) (layer F.Fab)
       (effects (font (size 0.5 0.5) (thickness 0.015)))
     )
@@
   )
   (module Capacitors_SMD:C_0805_HandSoldering (layer F.Cu)
-    (at 457.2 158.75 90)
+    (at 457.2 155.829 270)
     (descr "Capacitor SMD 0805, hand soldering")
     (tags "capacitor 0805")
     (attr smd)
-    (fp_text reference C_PW_BYNEG1 (at 0 -2.1 90) (layer F.SilkS)
-      (effects (font (size 0.5 0.5) (thickness 0.015)))
-    )
-    (fp_text value 100nF (at 0 2.1 90) (layer F.Fab)
+    (fp_text reference C_PW_BYNEG1 (at 0 -2.1 270) (layer F.SilkS)
+      (effects (font (size 0.5 0.5) (thickness 0.015)))
+    )
+    (fp_text value 100nF (at 0 2.1 270) (layer F.Fab)
       (effects (font (size 0.5 0.5) (thickness 0.015)))
     )
@@
     (fp_line (start 0.5 -0.85) (end -0.5 -0.85) (layer F.SilkS) (width 0.15))
     (fp_line (start -0.5 0.85) (end 0.5 0.85) (layer F.SilkS) (width 0.15))
-    (pad 1 smd rect (at -1.25 0 90) (size 1.5 1.25) (layers F.Cu F.Paste F.Mask)
-      (net 1 /GND))
-    (pad 2 smd rect (at 1.25 0 90) (size 1.5 1.25) (layers F.Cu F.Paste F.Mask)
+    (pad 1 smd rect (at -1.25 0 270) (size 1.5 1.25) (layers F.Cu F.Paste F.Mask)
+      (net 1 /GND))
+    (pad 2 smd rect (at 1.25 0 270) (size 1.5 1.25) (layers F.Cu F.Paste F.Mask)
       (net 2 /12V-))
     (model Capacitors_SMD.3dshapes/C_0805_HandSoldering.wrl
@@
   )
   (module Capacitors_SMD:C_0805_HandSoldering (layer F.Cu)
-    (at 457.2 146.05 90)
+    (at 457.2 148.844 270)
     (descr "Capacitor SMD 0805, hand soldering")
     (tags "capacitor 0805")
     (attr smd)
-    (fp_text reference C_PW_BYPOS1 (at 0 -2.1 90) (layer F.SilkS)
-      (effects (font (size 0.5 0.5) (thickness 0.015)))
-    )
-    (fp_text value 100nF (at 0 2.1 90) (layer F.Fab)
+    (fp_text reference C_PW_BYPOS1 (at 0 -2.1 270) (layer F.SilkS)
+      (effects (font (size 0.5 0.5) (thickness 0.015)))
+    )
+    (fp_text value 100nF (at 0 2.1 270) (layer F.Fab)
       (effects (font (size 0.5 0.5) (thickness 0.015)))
     )
@@
     (fp_line (start 0.5 -0.85) (end -0.5 -0.85) (layer F.SilkS) (width 0.15))
     (fp_line (start -0.5 0.85) (end 0.5 0.85) (layer F.SilkS) (width 0.15))
-    (pad 1 smd rect (at -1.25 0 90) (size 1.5 1.25) (layers F.Cu F.Paste F.Mask)
+    (pad 1 smd rect (at -1.25 0 270) (size 1.5 1.25) (layers F.Cu F.Paste F.Mask)
       (net 3 /12V+))
-    (pad 2 smd rect (at 1.25 0 90) (size 1.5 1.25) (layers F.Cu F.Paste F.Mask)
+    (pad 2 smd rect (at 1.25 0 270) (size 1.5 1.25) (layers F.Cu F.Paste F.Mask)
       (net 1 /GND))
     (model Capacitors_SMD.3dshapes/C_0805_HandSoldering.wrl
@@
       (effects (font (size 0.5 0.5) (thickness 0.015)))
     )
-    (fp_text value B100K (at 0 -6.604 90) (layer F.Fab)
+    (fp_text value B50K (at 0 -6.604 90) (layer F.Fab)
       (effects (font (size 0.5 0.5) (thickness 0.015)))
     )
@@
       (effects (font (size 0.5 0.5) (thickness 0.015)))
     )
-    (fp_text value B100K (at 0 -6.604 90) (layer F.Fab)
+    (fp_text value B5K (at 0 -6.604 90) (layer F.Fab)
       (effects (font (size 0.5 0.5) (thickness 0.015)))
     )
@@
       (effects (font (size 0.5 0.5) (thickness 0.015)))
     )
-    (fp_text value B100K (at 0 -6.604 90) (layer F.Fab)
+    (fp_text value B50K (at 0 -6.604 90) (layer F.Fab)
       (effects (font (size 0.5 0.5) (thickness 0.015)))
     )
@@
       (effects (font (size 0.5 0.5) (thickness 0.015)))
     )
-    (fp_text value B100K (at 0 -6.604 90) (layer F.Fab)
+    (fp_text value B5K (at 0 -6.604 90) (layer F.Fab)
       (effects (font (size 0.5 0.5) (thickness 0.015)))
     )
@@
       (effects (font (size 0.5 0.5) (thickness 0.015)))
     )
-    (fp_text value B100K (at 0 -6.604 90) (layer F.Fab)
+    (fp_text value B50K (at 0 -6.604 90) (layer F.Fab)
       (effects (font (size 0.5 0.5) (thickness 0.015)))
     )
@@
       (effects (font (size 0.5 0.5) (thickness 0.015)))
     )
-    (fp_text value B100K (at 0 -6.604 90) (layer F.Fab)
+    (fp_text value B50K (at 0 -6.604 90) (layer F.Fab)
       (effects (font (size 0.5 0.5) (thickness 0.015)))
     )
@@
       (effects (font (size 0.5 0.5) (thickness 0.015)))
     )
-    (fp_text value B100K (at 0 -6.604 90) (layer F.Fab)
+    (fp_text value B50K (at 0 -6.604 90) (layer F.Fab)
       (effects (font (size 0.5 0.5) (thickness 0.015)))
     )
@@
       (effects (font (size 0.5 0.5) (thickness 0.015)))
     )
-    (fp_text value B100K (at 0 -6.604 90) (layer F.Fab)
+    (fp_text value B50K (at 0 -6.604 90) (layer F.Fab)
       (effects (font (size 0.5 0.5) (thickness 0.015)))
     )
@@
     (pad 1 thru_hole rect (at 0 0) (size 1.7 1.7) (drill 1) (layers *.Cu *.Mask)
       (net 3 /12V+))
-    (pad 2 thru_hole oval (at 2.54 0) (size 1.7 1.7) (drill 1) (layers *.Cu *.Mask))
-    (pad 3 thru_hole oval (at 0 2.54) (size 1.7 1.7) (drill 1) (layers *.Cu *.Mask))
-    (pad 4 thru_hole oval (at 2.54 2.54) (size 1.7 1.7) (drill 1) (layers *.Cu *.Mask))
+    (pad 2 thru_hole oval (at 2.54 0) (size 1.7 1.7) (drill 1) (layers *.Cu *.Mask)
+      (net 44 "Net-(J_PWR1-Pad2)"))
+    (pad 3 thru_hole oval (at 0 2.54) (size 1.7 1.7) (drill 1) (layers *.Cu *.Mask)
+      (net 45 "Net-(J_PWR1-Pad3)"))
+    (pad 4 thru_hole oval (at 2.54 2.54) (size 1.7 1.7) (drill 1) (layers *.Cu *.Mask)
+      (net 46 "Net-(J_PWR1-Pad4)"))
     (pad 5 thru_hole oval (at 0 5.08) (size 1.7 1.7) (drill 1) (layers *.Cu *.Mask)
       (net 1 /GND))
-    (pad 6 thru_hole oval (at 2.54 5.08) (size 1.7 1.7) (drill 1) (layers *.Cu *.Mask))
-    (pad 7 thru_hole oval (at 0 7.62) (size 1.7 1.7) (drill 1) (layers *.Cu *.Mask))
-    (pad 8 thru_hole oval (at 2.54 7.62) (size 1.7 1.7) (drill 1) (layers *.Cu *.Mask))
+    (pad 6 thru_hole oval (at 2.54 5.08) (size 1.7 1.7) (drill 1) (layers *.Cu *.Mask)
+      (net 47 "Net-(J_PWR1-Pad6)"))
+    (pad 7 thru_hole oval (at 0 7.62) (size 1.7 1.7) (drill 1) (layers *.Cu *.Mask)
+      (net 48 "Net-(J_PWR1-Pad7)"))
+    (pad 8 thru_hole oval (at 2.54 7.62) (size 1.7 1.7) (drill 1) (layers *.Cu *.Mask)
+      (net 49 "Net-(J_PWR1-Pad8)"))
     (pad 9 thru_hole oval (at 0 10.16) (size 1.7 1.7) (drill 1) (layers *.Cu *.Mask)
       (net 2 /12V-))
-    (pad 10 thru_hole oval (at 2.54 10.16) (size 1.7 1.7) (drill 1) (layers *.Cu *.Mask))
+    (pad 10 thru_hole oval (at 2.54 10.16) (size 1.7 1.7) (drill 1) (layers *.Cu *.Mask)
+      (net 50 "Net-(J_PWR1-Pad10)"))
     (model ${KISYS3DMOD}/Pin_Headers.3dshapes/Pin_Header_Straight_2x05_Pitch2.54mm.wrl
       (at (xyz 0 0 0))

Commit message: First draft board layout
Parts:
- added R_ChanA_OAout1: 1K, Resistors_SMD:R_0805_HandSoldering, F.Cu at (442.6, 97.8)
- added R_ChanB_OAout1: 1K, Resistors_SMD:R_0805_HandSoldering, F.Cu at (483.9, 97.8)
- J_ChanA_out1, J_ChanB_out1, J_IN1, J_IN2, J_IN3, J_IN4, J_IN5, J_IN6, J_IN7, J_IN8: footprint ThonkiConn_3:Conn_3.5mmJackMono_Vertical_PJ301BM -> ThonkiConn_3:Conn_3.5mmJackMono_Vertical_PJ301M-12
- moved J_ChanA_out1 85.3 mm to (432.6, 86.4), turned to 180 degrees
- moved J_ChanB_out1 84.2 mm to (473.2, 86.4), turned to 180 degrees
- moved R_LED8 83.0 mm to (382.3, 102.9)
- moved C_PW_BYPOS1 79.5 mm to (411.5, 83.8), turned to 0 degrees
- moved J_PWR1 77.2 mm to (410.2, 93.3)
- moved VR_FADER8 76.8 mm to (390.5, 97.8)
- moved R_LED7 76.6 mm to (341.6, 103.0)
- moved R_ChanA_OAout_Rin1 76.1 mm to (428.0, 105.4)
- moved C_ChanA_POSBY1 76.0 mm to (433.7, 97.8)
- moved U_ChanA_OA1 75.6 mm to (435.6, 105.4)
- moved C_ChanA_NEGBY1 75.2 mm to (437.5, 113.0)
- moved VR_ChanA_OAout_Rf1 74.8 mm to (451.5, 97.8)
- moved C_ChanB_BYPOS1 74.4 mm to (474.3, 97.8)
- moved R_ChanA_OAin_Rf1 74.3 mm to (429.3, 111.8)
- moved U_ChanB_OA1 74.0 mm to (476.2, 105.4)
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Connections:
- VR_ChanA_OAout_Rf1 pad 4: (no net) -> /12V+
- VR_ChanA_OAout_Rf1 pad 5: (no net) -> Net-(R_ChanA_OAout1-Pad1)
- VR_ChanB_OAout_Rf1 pad 4: (no net) -> /12V+
- VR_ChanB_OAout_Rf1 pad 5: (no net) -> Net-(R_ChanB_OAout1-Pad1)
Routing:
- net /12V+: track 0.00 -> 509.1 mm
- net Net-(R_ChanB_OAin_Rf1-Pad2): track 0.00 -> 447.9 mm, vias 0 -> 2
- net Net-(R_ChanA_OAin_Rf1-Pad2): track 0.00 -> 387.4 mm, vias 0 -> 1
- net /12V-: track 0.00 -> 93.1 mm
- net Net-(R_ChanB_OAout_Rin1-Pad1): track 0.00 -> 78.6 mm
- net Net-(R_ChanA_OAout_Rin1-Pad1): track 0.00 -> 77.9 mm
- net /GND: track 0.00 -> 46.8 mm, vias 0 -> 21
- net Net-(J_ChanA_out1-Pad3): track 0.00 -> 37.7 mm
- net Net-(J_ChanB_out1-Pad3): track 0.00 -> 37.1 mm
- net Net-(J_IN7-Pad3): track 0.00 -> 33.8 mm
- net Net-(J_IN3-Pad3): track 0.00 -> 33.8 mm
- net Net-(J_IN6-Pad3): track 0.00 -> 33.8 mm
- net Net-(J_IN2-Pad3): track 0.00 -> 33.8 mm
- net Net-(J_IN5-Pad3): track 0.00 -> 33.4 mm
- net Net-(J_IN4-Pad3): track 0.00 -> 33.4 mm
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- added copper zone on B.Cu, net /GND
Other:
- board size 478.8 x 43.2 mm -> 426.7 x 43.2 mm
- board text added: "+12V"
- board text added: "-12V"
- board text added: "1"
- board text added: "2"
- board text added: "3"
- board text added: "4"
- board text added: "5"
- board text added: "6"
- board text added: "7"
- board text added: "8"
- board text added: "A"
- board text added: "B"
- board text added: "GND"

Commit message: second draft
Parts:
- added REF**: MountingHole_3.2mm_M3, Mounting_Holes:MountingHole_3.2mm_M3, F.Cu at (84.0, 79.2)
- added REF**: MountingHole_3.2mm_M3, Mounting_Holes:MountingHole_3.2mm_M3, F.Cu at (84.0, 116.4)
- added REF**: MountingHole_3.2mm_M3, Mounting_Holes:MountingHole_3.2mm_M3, F.Cu at (495.7, 116.4)
- added REF**: MountingHole_3.2mm_M3, Mounting_Holes:MountingHole_3.2mm_M3, F.Cu at (495.7, 79.2)
- moved R_LED1 20.3 mm to (97.1, 82.6)
- moved R_LED8 20.3 mm to (381.6, 82.5)
- moved R_LED2 20.3 mm to (138.3, 82.6)
- moved R_LED3 20.3 mm to (179.1, 82.5)
- moved R_LED4 20.3 mm to (219.7, 82.5)
- moved R_LED5 20.3 mm to (260.3, 82.6)
- moved R_LED6 20.3 mm to (300.9, 82.6)
- moved R_LED7 20.3 mm to (341.6, 82.6)
- moved R_ChanB_OAout1 13.7 mm to (483.9, 84.1)
- moved R_ChanA_OAout1 13.6 mm to (443.2, 84.2)
- turned VR_ChanA_OAout_Rf1 to 270 degrees
- turned VR_ChanB_OAout_Rf1 to 270 degrees
- turned VR_FADER1 to 270 degrees
- turned VR_FADER2 to 270 degrees
- turned VR_FADER3 to 270 degrees
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Routing:
- net /12V+: track 509.1 -> 847.9 mm
- net Net-(R_ChanA_OAout_Rin1-Pad1): track 77.9 -> 37.4 mm
- net Net-(R_ChanB_OAout_Rin1-Pad1): track 78.6 -> 38.6 mm
- net Net-(R_ChanA_OAout1-Pad1): track 23.8 -> 4.55 mm
- net Net-(R_ChanB_OAout1-Pad1): track 22.9 -> 4.43 mm
- net Net-(R_LED8-Pad1): track 18.7 -> 4.00 mm
- net Net-(R_LED2-Pad1): track 17.7 -> 3.41 mm
- net Net-(R_LED3-Pad1): track 17.6 -> 3.36 mm
- net Net-(R_LED7-Pad1): track 17.3 -> 3.41 mm
- net Net-(R_LED6-Pad1): track 17.3 -> 3.41 mm
- net Net-(R_LED5-Pad1): track 16.9 -> 3.41 mm
- net Net-(R_ChanAB_OAin_Rin4-Pad2): track 26.0 -> 39.5 mm
- net Net-(R_ChanAB_OAin_Rin5-Pad2): track 25.5 -> 39.0 mm
- net Net-(R_ChanAB_OAin_Rin7-Pad2): track 25.9 -> 39.4 mm
- net Net-(R_LED4-Pad1): track 16.5 -> 3.36 mm
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Other:
- board size 426.7 x 43.2 mm -> 426 x 43.2 mm

Commit message: third draft
Parts:
- moved R_ChanAB_OAin_Rin2 5.00 mm to (129.5, 101.6)
- moved J_IN1 5.00 mm to (92.0, 86.4)
- moved J_IN2 5.00 mm to (132.8, 86.4)
- moved J_IN3 5.00 mm to (173.4, 86.4)
- moved J_IN4 5.00 mm to (214.0, 86.4)
- moved J_IN5 5.00 mm to (254.7, 86.4)
- moved J_IN6 5.00 mm to (295.3, 86.4)
- moved J_IN7 5.00 mm to (335.8, 86.4)
- moved J_IN8 5.00 mm to (376.6, 86.4)
- moved R_ChanAB_OAin_Rin1 5.00 mm to (88.8, 101.6)
- moved R_ChanAB_OAin_Rin3 5.00 mm to (170.1, 101.6)
- moved R_ChanAB_OAin_Rin4 5.00 mm to (210.7, 101.6)
- moved R_ChanAB_OAin_Rin5 5.00 mm to (251.4, 101.6)
- moved R_ChanAB_OAin_Rin6 5.00 mm to (292.0, 101.6)
- moved R_ChanAB_OAin_Rin7 5.00 mm to (332.7, 101.5)
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Routing:
- net /12V+: track 847.9 -> 823.6 mm
- net Net-(R_ChanB_OAin_Rf1-Pad2): track 447.9 -> 425.7 mm, vias 2 -> 1
- net Net-(J_ChanB_out1-Pad3): track 49.9 -> 37.0 mm
- net Net-(R_ChanA_OAout_Rin1-Pad1): track 37.4 -> 27.2 mm
- net Net-(J_ChanA_out1-Pad3): track 47.6 -> 38.1 mm
- net Net-(R_ChanB_OAout_Rin1-Pad1): track 38.6 -> 29.5 mm
- net Net-(R_ChanAB_OAin_Rin4-Pad2): track 39.5 -> 33.2 mm
- net Net-(R_ChanAB_OAin_Rin7-Pad2): track 39.4 -> 33.2 mm
- net Net-(R_ChanAB_OAin_Rin6-Pad2): track 39.0 -> 33.2 mm
- net Net-(R_ChanAB_OAin_Rin5-Pad2): track 39.0 -> 33.2 mm
- net /GND: track 47.4 -> 41.7 mm, vias 21 -> 20
- net Net-(R_ChanAB_OAin_Rin2-Pad2): track 37.5 -> 33.2 mm
- net Net-(R_ChanAB_OAin_Rin3-Pad2): track 37.5 -> 33.2 mm
- net Net-(R_ChanAB_OAin_Rin1-Pad2): track 37.2 -> 33.2 mm
- net Net-(R_ChanA_OAin_Rf1-Pad2): track 387.4 -> 390.9 mm
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
Commit message: minor updates
Parts:
- moved C_PW_BYPOS1 6.12 mm to (410.8, 87.6), turned to 90 degrees
- moved C_PW_BYNEG1 5.90 mm to (411.0, 108.2), turned to 90 degrees
Routing:
- net /12V-: track 91.4 -> 84.1 mm
- net /12V+: track 823.6 -> 818.7 mm
