File: 1URack_8Input_AB_2Output_Mixer.kicad_pcb (KiCad board)
At the start: 2 copper layers, 426 x 43.2 mm, 63 parts

Commit message: updated to Kicad 5
Parts:
- removed REF** (x4): MountingHole_3.2mm_M3, Mounting_Holes:MountingHole_3.2mm_M3
- R_ChanA_OAout_Rin1, R_ChanB_OAout_Rin1: value 25K -> 22K
- R_LED1, R_LED2, R_LED3, R_LED4, R_LED5, R_LED6, R_LED7, R_LED8: value 560R -> 2K2
