File: FrontPanel/FrontPanel_1URack_8Input_AB_2Output_Mixer.kicad_pcb (KiCad board)
At the start: 2 copper layers, 426 x 43.2 mm, 22 parts

Commit message: Created Front Panel REVB
Parts:
- removed the REF** at (495.7, 116.4)
- removed the REF** at (84.0, 116.3)
- removed the REF** at (495.7, 79.2)
- removed the REF** at (84.0, 79.2)
- added REF**: MountingHole_5.3mm_M5_ISO14580, MountingHole:MountingHole_5.3mm_M5_ISO14580, F.Cu at (54.6, 81.9)
- added REF**: MountingHole_5.3mm_M5_ISO14580, MountingHole:MountingHole_5.3mm_M5_ISO14580, F.Cu at (54.6, 113.7)
- added REF**: MountingHole_5.3mm_M5_ISO14580, MountingHole:MountingHole_5.3mm_M5_ISO14580, F.Cu at (524.5, 113.5)
- added REF**: MountingHole_5.3mm_M5_ISO14580, MountingHole:MountingHole_5.3mm_M5_ISO14580, F.Cu at (524.5, 82.0)
- REF** (x8): value MountingHole_4.5mm -> MountingHole_5.3mm_M5_ISO14580; footprint MountingHole:MountingHole_4.5mm -> MountingHole:MountingHole_5.3mm_M5_ISO14580
- REF** (x10): value MountingHole_4.5mm -> MountingHole_6.4mm_M6_ISO14580; footprint MountingHole:MountingHole_4.5mm -> MountingHole:MountingHole_6.4mm_M6_ISO14580
Routing:
- removed copper zone on B.Cu, net /GND
Other:
- board size 426 x 43.2 mm -> 481.3 x 43.2 mm
- board text added: "OFF"
