File: Hardware/1URack_8Input_AB_2Output_Mixer.sch (KiCad schematic (older format))
At the start: 59 parts

Commit message: Documentation corrections and restructure
Parts:
- VR_FADER2, VR_FADER4: value B5K -> B50K
Changed lines of the file:
@@
 P 2900 6475
 F 0 "VR_FADER2" H 3150 6725 50  0000 C CNN
-F 1 "B5K" H 3150 6625 50  0000 C CNN
+F 1 "B50K" H 3150 6625 50  0000 C CNN
 F 2 "Bourn_PTL_Slider:Slider_PTL20_LED_35MM" H 2900 6475 50  0001 C CNN
 F 3 "" H 2900 6475 50  0001 C CNN
@@
 P 2900 9775
 F 0 "VR_FADER4" H 3125 10050 50  0000 C CNN
-F 1 "B5K" H 3125 9975 50  0000 C CNN
+F 1 "B50K" H 3125 9975 50  0000 C CNN
 F 2 "Bourn_PTL_Slider:Slider_PTL20_LED_35MM" H 2900 9775 50  0001 C CNN
 F 3 "" H 2900 9775 50  0001 C CNN
